Commit message: :zap: update pid parameters

File: gym_quad/assets/cf2x.urdf (robot description, URDF)
Before this commit: robot cf2, 2 links, 1 joints
Links:
- added link rope_end, mass 0.01; collision sphere radius=.01; visual sphere radius=.01
- added link virtual_link0, mass 0
Joints:
- added joint joint0_x: type revolute, parent center_of_mass_link, child virtual_link0, origin xyz=0 0 0.0 rpy=0 0 0, axis 1 0 0, limit lower=-10000 upper=10000 effort=1000.0 velocity=1000.0
- added joint joint0_y: type revolute, parent virtual_link0, child rope_end, origin xyz=0 0 0.0 rpy=0 0 0, axis 0 1 0, limit lower=-10000 upper=10000 effort=1000.0 velocity=1000.0

Commit message: :zap: add hangging objects

File: gym_quad/assets/cf2x.urdf (robot description, URDF)
Before this commit: robot cf2, 4 links, 3 joints
Links:
- added link hook, mass 0
Joints:
- added joint hook_joint: type fixed, parent center_of_mass_link, child hook, origin xyz=0.0 0.0 -0.03 rpy=0.00000 -0.00000 0.00000, axis 0.00000 0.00000 0.00000
- joint joint0_x: origin xyz=0 0 0.0 rpy=0 0 0 -> xyz=0.0 0.0 0.0 rpy=0 0 0; parent center_of_mass_link -> hook
- joint joint0_y: origin xyz=0 0 0.0 rpy=0 0 0 -> xyz=0 0 0 rpy=0 0 0

Commit message: :zap: update readme with TODO list

File: gym_quad/assets/cf2x.urdf (robot description, URDF)
Before this commit: robot cf2, 5 links, 4 joints
Links:
- link rope_end: mass 0.01 -> 0.00001

File: gym_quad/assets/cf2x_dual.urdf (robot description, URDF)
Before this commit: robot cf2_dual, 13 links, 12 joints
Links:
- link obj: mass 0.01 -> 0.00001

Commit message: :zap: bi-level PID controller for single agent transportation

File: gym_quad/assets/cf2x.urdf (robot description, URDF)
Before this commit: robot cf2, 5 links, 4 joints
Links:
- link rope_end: mass 0.00001 -> 0.01

Commit message: :zap: align with the torch-based environment.

File: gym_quad/assets/cf2x.urdf (robot description, URDF)
Before this commit: robot cf2, 5 links, 4 joints
Joints:
- joint hook_joint: origin xyz=0.0 0.0 -0.03 rpy=0.00000 -0.00000 0.00000 -> xyz=0.0 0.0 -0.05 rpy=0.00000 -0.00000 0.00000

Commit message: :sparkles: add joint force sensor

File: gym_quad/assets/cf2x.urdf (robot description, URDF)
Before this commit: robot cf2, 5 links, 4 joints
Links:
- added link obj, mass 0.01; collision sphere radius=.01; visual sphere radius=.01
- link rope_end: mass 0.01 -> 0; geometry 
Joints:
- added joint obj_joint: type fixed, parent rope_end, child obj, origin xyz=0 0.0 0.0 rpy=0 0 0
