Commit message: fix index problem in cf2x_addrope.urdf

File: gym_quad/assets/cf2x_addrope.urdf (robot description, URDF)
Before this commit: robot cf2_add_rope, 6 links, 5 joints
Links:
- link link1: mass 0.0001 -> 0
- link link2: mass 0.0001 -> 0

Commit message: add rope v2

File: gym_quad/assets/cf2x_addrope.urdf (robot description, URDF)
Before this commit: robot cf2_add_rope, 6 links, 5 joints
Links:
- added link link3, mass 0; collision cylinder length=0.05 radius=0.0001; visual cylinder length=0.05 radius=0.0001
- link link2: geometry collision cylinder length=0.05 radius=0.0001; visual cylinder length=0.05 radius=0.0001
Joints:
- added joint joint3: type revolute, parent link2, child link3, origin xyz=0.0 0.0 -0.05 rpy=0 0 0, axis 1 1 0, limit lower=-10000 upper=10000 effort=1000.0 velocity=1000.0
- joint joint0_y: origin xyz=0 0 -0.09 rpy=0 0 0 -> xyz=0 0 -0.04 rpy=0 0 0; parent link2 -> link3

Commit message: fix dualquad urdf problems

File: gym_quad/assets/cf2x_addrope.urdf (robot description, URDF)
Before this commit: robot cf2_add_rope, 7 links, 6 joints
Joints:
- joint joint3: axis 1 1 0 -> 0 1 0

File: gym_quad/assets/cf2x_dual.urdf (robot description, URDF)
Before this commit: robot cf2_dual, 13 links, 12 joints
Links:
- link cf1_down: mass None -> 0.0
- link cf1_hook: mass None -> 0.0
- link cf1_mid: mass None -> 0.0
- link cf2_down: mass None -> 0.0
- link cf2_hook: mass None -> 0.0
- link cf2_mid: mass None -> 0.0
- link obj: mass 0.00001 -> 0.01
- link obj_left: mass None -> 0.0
- link obj_left_up: mass None -> 0.0; geometry visual cylinder length=0.21 radius=0.0001
- link obj_right: mass None -> 0.0
- link obj_right_up: mass None -> 0.0; geometry visual cylinder length=0.21 radius=0.0001
