Commit message: add triple version

File: gym_quad/assets/cf2x_triple.urdf (robot description, URDF)
Before this commit: robot cf2_dual, 13 links, 12 joints
Links:
- added link cf3, mass 0.027; collision cylinder length=.025 radius=.06; visual mesh filename=./cf2.dae scale=1 1 1
- added link cf3_down, mass 0.0
- added link cf3_hook, mass 0.0
- added link cf3_mid, mass 0.0
- added link obj_back, mass 0.0
- added link obj_back_up, mass 0.0
Joints:
- added joint cf3_fixed: type fixed, parent cf3_hook, child cf3, origin xyz=0.0 0.0 0.03 rpy=0.00000 -0.00000 0.00000, axis 0.00000 0.00000 0.00000
- added joint cf3_x: type revolute, parent cf3_down, child cf3_mid, origin xyz=0.0 0.0 0.0 rpy=0 0 0, axis 1 0 0, limit lower=-10000 upper=10000 effort=1000.0 velocity=1000.0
- added joint cf3_y: type revolute, parent cf3_mid, child cf3_hook, origin xyz=0.0 0.0 0.0 rpy=0 0 0, axis 0 1 0, limit lower=-10000 upper=10000 effort=1000.0 velocity=1000.0
- added joint obj_back_up_joint: type fixed, parent obj_back_up, child cf3_down, origin xyz=0 -0.2 0.2828 rpy=0.00000 -0.00000 0.00000, axis 0.00000 0.00000 0.00000
- added joint obj_back_x: type fixed, parent obj, child obj_back, origin xyz=0.0 0.0 0.0 rpy=0 0 0, axis 1 0 0, limit lower=-10000 upper=10000 effort=1000.0 velocity=1000.0
- added joint obj_back_y: type fixed, parent obj_back, child obj_back_up, origin xyz=0.0 0.0 0.0 rpy=0 0 0, axis 0 1 0, limit lower=-10000 upper=10000 effort=1000.0 velocity=1000.0
- joint obj_left_up_joint: origin xyz=0.15 0.0 0.15 rpy=0.00000 -0.00000 0.00000 -> xyz=0.1732 0.1 0.2828 rpy=0.00000 -0.00000 0.00000
- joint obj_right_up_joint: origin xyz=-0.15 0.0 0.15 rpy=0.00000 -0.00000 0.00000 -> xyz=-0.1732 0.1 0.2828 rpy=0.00000 -0.00000 0.00000
